File: Hardware/Eagle/TempestDrone2_V3/TempestDrone2.sch (EAGLE design)
At the start: 45 parts, among them CON1 MOLEX_51281-1094, CON2 B2B-ZR(LF)(SN), CON3 20021111-00010T4LF, CON4 USB-MICRO-A, CON5 M50-3000545, IC1 ATSAMD21E17A-MU, Q1 dnp, SW3 B3U-1000P, U1 TPS70933DBVR

Commit message: - Minor improvements
Parts:
- removed SW3: B3U-1000P, squirrel:PUSHBUTTONMICRO2
- added S4: SWITCH-MOMENTARY-2B3U-1000P, squirrel:SWITCH-MOMENTARY-2B3U-1000P
- CON1: PART# (none) -> 51281-1094; SUPP (none) -> Molex
- CON2: PART# (none) -> B2B-ZR(LF)(SN); SUPP (none) -> JST
- CON3: PART# (none) -> 20021111-00010T4LF; SUPP (none) -> FCI
- CON5: value M50-3000545 -> M50-3000545 (alt. GRPB052VWVN-RC); PART# (none) -> M50-3000545; SUPP (none) -> Harwin
- IC1: PART# (none) -> ATSAMD21E17A-MU; SUPP (none) -> Atmel
- LED1: value LTST-S310F2KT -> LTST-S310F2KT (alt 5988810307F or OVSRRGBCC3); PART# (none) -> LTST-S310F2KT; SUPP (none) -> Lite-On
- S1, S2: PART# (none) -> 1-1825027-1; SUPP (none) -> TE
- S3: PART# (none) -> D2F-L-A; SUPP (none) -> Omron
- U$1: value AMS002 -> AMS001/AMS002; PART# (none) -> AMS001 or AMS002; SUPP (none) -> Zentri/ack.me
- U1: PART# (none) -> TPS70933DBVR; SUPP (none) -> TI
Connections:
- net GND: now also S4.2; no longer SW3.2, SW3.2A
- net TOUR_BUT: now also S4.1; no longer SW3.1, SW3.1A
