File: Hardware/Eagle/TempestDrone2_V3/TempestDrone2.brd (EAGLE design)
At the start: 35.2 x 86.5 mm, 45 parts, among them CON1 MOLEX_51281-1094, CON2 B2B-ZR(LF)(SN), CON3 20021111-00010T4LF, CON4 USB-MICRO-A, CON5 M50-3000545, IC1 ATSAMD21E17A-MU, Q1 dnp, SW3 B3U-1000P, U1 TPS70933DBVR

Commit message: - Minor improvements
Parts:
- removed SW3: B3U-1000P, squirrel:PUSHBUTTON-MICRO2
- added S4: SWITCH-MOMENTARY-2B3U-1000P, squirrel:PUSHBUTTON-MICRO3
- CON5: value M50-3000545 -> M50-3000545 (alt. GRPB052VWVN-RC)
- LED1: value LTST-S310F2KT -> LTST-S310F2KT (alt 5988810307F or OVSRRGBCC3)
- U$1: value AMS002 -> AMS001/AMS002
Connections:
- net GND: now also S4.2A; no longer SW3.2A, SW3.2B
- net TOUR_BUT: now also S4.1A; no longer SW3.1A, SW3.1B
Routing:
- net N$7: track 57.2 -> 56.1 mm
- net TOUR_BUT: track 21.6 -> 21.1 mm
- net GND: track 39.8 -> 39.6 mm, vias 37 -> 39

Commit message: - New Shocker upper board for Luxe solenoid - Update of lib
Routing:
- net GND: vias 39 -> 38
Changed lines of the file:
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@@
 <layer number="19" name="Unrouted" color="6" fill="1" visible="yes" active="yes"/>
 <layer number="20" name="Dimension" color="15" fill="1" visible="yes" active="yes"/>
-<layer number="21" name="tPlace" color="7" fill="1" visible="yes" active="yes"/>
-<layer number="22" name="bPlace" color="7" fill="1" visible="yes" active="yes"/>
+<layer number="21" name="tPlace" color="7" fill="1" visible="no" active="yes"/>
+<layer number="22" name="bPlace" color="7" fill="1" visible="no" active="yes"/>
 <layer number="23" name="tOrigins" color="15" fill="1" visible="yes" active="yes"/>
-<layer number="24" name="bOrigins" color="15" fill="1" visible="yes" active="yes"/>
-<layer number="25" name="tNames" color="7" fill="1" visible="yes" active="yes"/>
-<layer number="26" name="bNames" color="7" fill="1" visible="yes" active="yes"/>
-<layer number="27" name="tValues" color="7" fill="1" visible="no" active="yes"/>
+<layer number="24" name="bOrigins" color="15" fill="1" visible="no" active="yes"/>
+<layer number="25" name="tNames" color="7" fill="1" visible="no" active="yes"/>
+<layer number="26" name="bNames" color="7" fill="1" visible="no" active="yes"/>
+<layer number="27" name="tValues" color="7" fill="1" visible="yes" active="yes"/>
 <layer number="28" name="bValues" color="7" fill="1" visible="no" active="yes"/>
 <layer number="29" name="tStop" color="7" fill="3" visible="no" active="yes"/>
@@
 <layer number="50" name="dxf" color="7" fill="1" visible="no" active="yes"/>
 <layer number="51" name="tDocu" color="7" fill="1" visible="yes" active="yes"/>
-<layer number="52" name="bDocu" color="7" fill="1" visible="yes" active="yes"/>
+<layer number="52" name="bDocu" color="7" fill="1" visible="no" active="yes"/>
 <layer number="53" name="tGND_GNDA" color="7" fill="1" visible="no" active="yes"/>
 <layer number="54" name="bGND_GNDA" color="7" fill="1" visible="no" active="yes"/>
@@
 <contactref element="S4" pad="2A"/>
 <via x="34.1" y="57" extent="1-16" drill="0.3"/>
-<via x="34.1" y="54.4" extent="1-16" drill="0.3"/>
 </signal>
 <signal name="VCC">
