File: Hardware/Eagle/Tempest/Tempest.sch (EAGLE design)
At the start: 62 parts, among them CON1 B3B-ZR, CON2 B2B-ZR, CON3 B4B-ZR, CON4 HDR2MM-8, CON5 HDR2MM-8, CON6 USB-MICRO-A, CON7 FE05-2HD-2, IC1 ATSAMD21E, IC2 MMA8652, IC3 TPS62150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

Commit message: - Added 100K between power button and controller - Added part # for fets and diodes
Parts:
- added R17: 100k, squirrel:R0603
- D1, D2, D6: value SOD123 -> PMEG4010ETR
- D4: value (none) -> BZT52C20
- T1, T2: value (none) -> ZXMN3A03E6
Connections:
- new net N$8: R17.1, SW1.1
- net SAM_SW: now also R17.2; no longer SW1.1
Changed lines of the file:
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@@
 </classes>
 <parts>
-<part name="T1" library="squirrel" deviceset="NMOSSOT23-6" device=""/>
-<part name="T2" library="squirrel" deviceset="NMOSSOT23-6" device=""/>
+<part name="T1" library="squirrel" deviceset="NMOSSOT23-6" device="" value="ZXMN3A03E6"/>
+<part name="T2" library="squirrel" deviceset="NMOSSOT23-6" device="" value="ZXMN3A03E6"/>
 <part name="C14" library="squirrel" deviceset="C-EU" device="C1206" value="10µ"/>
 <part name="C15" library="squirrel" deviceset="C-EU" device="C1206" value="22µ"/>
@@
 <part name="GND5" library="squirrel" deviceset="GND" device=""/>
 <part name="GND6" library="squirrel" deviceset="GND" device=""/>
-<part name="D1" library="squirrel" deviceset="DIODE-SCHOTTKY" device="SOD123" value="SOD123"/>
-<part name="D2" library="squirrel" deviceset="DIODE-SCHOTTKY" device="SOD123" value="SOD123"/>
-<part name="D4" library="squirrel" deviceset="ZENER-DIODE" device="SOD123"/>
-<part name="D6" library="squirrel" deviceset="DIODE-SCHOTTKY" device="SOD123" value="SOD123"/>
+<part name="D1" library="squirrel" deviceset="DIODE-SCHOTTKY" device="SOD123" value="PMEG4010ETR"/>
+<part name="D2" library="squirrel" deviceset="DIODE-SCHOTTKY" device="SOD123" value="PMEG4010ETR"/>
+<part name="D4" library="squirrel" deviceset="ZENER-DIODE" device="SOD123" value="BZT52C20"/>
+<part name="D6" library="squirrel" deviceset="DIODE-SCHOTTKY" device="SOD123" value="PMEG4010ETR"/>
 <part name="CON4" library="squirrel" deviceset="HDR2MM-8" device=""/>
 <part name="P+4" library="squirrel" deviceset="V+" device="" value="V9_PROT"/>
@@
 <part name="FID5" library="squirrel" deviceset="FIDUCIAL" device="UFIDUCIAL"/>
 <part name="FID6" library="squirrel" deviceset="FIDUCIAL" device="UFIDUCIAL"/>
+<part name="R17" library="squirrel" deviceset="R" device="0603" value="100k"/>
 </parts>
 <sheets>
@@
 <instance part="FID2" gate="G$1" x="17.78" y="241.3"/>
 <instance part="FID6" gate="G$1" x="17.78" y="233.68"/>
+<instance part="R17" gate="&gt;NAME" x="246.38" y="50.8" rot="R180"/>
 </instances>
 <busses>
@@
 <label x="226.06" y="50.8" size="1.778" layer="95"/>
 <wire x1="226.06" y1="50.8" x2="238.76" y2="50.8" width="0.1524" layer="91"/>
-<wire x1="238.76" y1="50.8" x2="254" y2="50.8" width="0.1524" layer="91"/>
-<pinref part="SW1" gate="SW" pin="1"/>
-<wire x1="254" y1="50.8" x2="261.62" y2="50.8" width="0.1524" layer="91"/>
+<wire x1="238.76" y1="50.8" x2="241.3" y2="50.8" width="0.1524" layer="91"/>
+<pinref part="R17" gate="&gt;NAME" pin="2"/>
 </segment>
 <segment>
@@
 </segment>
 </net>
+<net name="N$8" class="0">
+<segment>
+<pinref part="SW1" gate="SW" pin="1"/>
+<wire x1="254" y1="50.8" x2="261.62" y2="50.8" width="0.1524" layer="91"/>
+<wire x1="251.46" y1="50.8" x2="254" y2="50.8" width="0.1524" layer="91"/>
+<pinref part="R17" gate="&gt;NAME" pin="1"/>
+</segment>
+</net>
